Commit message: sync: release v0.1.1 from internal open_arm_sdk (64492db)

File: deps/zbl_arm_6a_description/share/zbl_arm_6a_description/urdf/parallel_gripper.ros2_control.xacro (robot description, xacro)
@@ -2,5 +2,5 @@
 <robot xmlns:xacro="http://www.ros.org/wiki/xacro">
   <xacro:macro name="parallel_gripper_ros2_control"
-               params="name prefix can_interface use_ipc:=1 mock_robot">
+               params="name prefix can_interface:=can0 use_ipc:=1 mock_robot domain:=0x04 unit:=0x00 auto_enable:=True">
     <ros2_control name="${name}"
                   type="system">
@@ -13,7 +13,10 @@
           <param name="can_interface">${can_interface}</param>
           <param name="use_ipc">${use_ipc}</param>
+          <param name="domain">${domain}</param>
+          <param name="unit">${unit}</param>
         </xacro:unless>
       </hardware>
       <joint name="${prefix}gripper">
+        <param name="auto_enable">${auto_enable}</param>
         <param name="motor_id">8</param>
         <param name="master_id">0</param>
@@ -21,4 +24,8 @@
         <param name="motor_hw_type">DM4310</param>
         <param name="max_torque">2.0</param>
+        <param name="lower_limit">0.0</param>
+        <param name="upper_limit">5.0</param>
+        <param name="default_kp">6.0</param>
+        <param name="default_kd">0.1</param>
         <param name="default_mode">tor</param>
         <command_interface name="position" />

File: deps/zbl_arm_6a_description/share/zbl_arm_6a_description/urdf/zbl_arm_6a.ros2_control.xacro (robot description, xacro)
@@ -2,5 +2,5 @@
 <robot xmlns:xacro="http://www.ros.org/wiki/xacro">
   <xacro:macro name="zbl_arm_6a_ros2_control"
-               params="name prefix can_interface use_ipc:=1 mock_robot">
+               params="name prefix can_interface:=can0 use_ipc:=1 mock_robot domain:=0x04 unit:=0x00 auto_enable:=True">
     <ros2_control name="${name}"
                   type="system">
@@ -13,7 +13,10 @@
           <param name="can_interface">${can_interface}</param>
           <param name="use_ipc">${use_ipc}</param>
+          <param name="domain">${domain}</param>
+          <param name="unit">${unit}</param>
         </xacro:unless>
       </hardware>
       <joint name="${prefix}arm_joint1">
+        <param name="auto_enable">${auto_enable}</param>
         <param name="motor_id">1</param>
         <param name="master_id">17</param>
@@ -33,4 +36,5 @@
       </joint>
       <joint name="${prefix}arm_joint2">
+        <param name="auto_enable">${auto_enable}</param>
         <param name="motor_id">2</param>
         <param name="master_id">18</param>
@@ -50,4 +54,5 @@
       </joint>
       <joint name="${prefix}arm_joint3">
+        <param name="auto_enable">${auto_enable}</param>
         <param name="motor_id">3</param>
         <param name="master_id">19</param>
@@ -68,4 +73,5 @@
       </joint>
       <joint name="${prefix}arm_joint4">
+        <param name="auto_enable">${auto_enable}</param>
         <param name="motor_id">4</param>
         <param name="master_id">20</param>
@@ -86,4 +92,5 @@
       </joint>
       <joint name="${prefix}arm_joint5">
+        <param name="auto_enable">${auto_enable}</param>
         <param name="motor_id">5</param>
         <param name="master_id">21</param>
@@ -104,4 +111,5 @@
       </joint>
       <joint name="${prefix}arm_joint6">
+        <param name="auto_enable">${auto_enable}</param>
         <param name="motor_id">6</param>
         <param name="master_id">22</param>

File: deps/zbl_arm_6a_description/share/zbl_arm_6a_description/urdf/zbl_arm_6a_with_gripper.xacro (robot description, xacro)
@@ -8,6 +8,18 @@
   <xacro:arg name="mock_robot"
              default="True" />
-  <!-- Add arx r5 arm -->
-  <xacro:include filename="$(find zbl_arm_6a_description)/urdf/zbl_arm_6a.urdf.xacro" />
+  <!-- Arm motor variant: hy (Huayi, default) or dm (DaMiao) -->
+  <xacro:arg name="arm_type" default="hy" />
+  <xacro:property name="arm_type_prop" value="$(arg arm_type)" />
+  <!-- Gripper variant: g (zbl g-gripper, default) or parallel (fx001 parallel gripper) -->
+  <xacro:arg name="gripper_type" default="g" />
+  <xacro:property name="gripper_type_prop" value="$(arg gripper_type)" />
+  <xacro:arg name="can_interface" default="can0" />
+  <!-- Add arx r5 arm: select URDF by arm_type -->
+  <xacro:if value="${arm_type_prop == 'hy'}">
+    <xacro:include filename="$(find zbl_arm_6a_description)/urdf/zbl_arm_6a_hy.urdf.xacro" />
+  </xacro:if>
+  <xacro:if value="${arm_type_prop == 'dm'}">
+    <xacro:include filename="$(find zbl_arm_6a_description)/urdf/zbl_arm_6a.urdf.xacro" />
+  </xacro:if>
   <xacro:zbl_arm_6a prefix=""
                         use_geometry_collision="$(arg use_geometry_collision)" />
@@ -22,23 +34,43 @@
   <xacro:zbl_arm_6a_ros2_control name="arm_control"
                                      prefix=""
-                                     can_interface="can0"
+                                     can_interface="$(arg can_interface)"
                                      use_ipc="1"
                                      mock_robot="$(arg mock_robot)" />
-  <!-- gripper -->
-  <xacro:include filename="$(find zbl_arm_6a_description)/urdf/parallel_gripper.urdf.xacro" />
-  <xacro:include filename="$(find zbl_arm_6a_description)/urdf/parallel_gripper.ros2_control.xacro" />
-  <xacro:parallel_gripper prefix="arm_"
-                                use_geometry_collision="$(arg use_geometry_collision)" />
-  <joint name="gripper_connector"
-         type="fixed">
-    <parent link="arm_link6" />
-    <child link="arm_gripper_base_link" />
-    <origin xyz="0 0 0"
-            rpy="0 0 0" />
-  </joint>
-  <xacro:parallel_gripper_ros2_control name="arm_gripper"
-                                             prefix="arm_"
-                                             can_interface="can0"
-                                             use_ipc="1"
-                                             mock_robot="$(arg mock_robot)" />
+  <!-- gripper: select by gripper_type -->
+  <xacro:if value="${gripper_type_prop == 'parallel'}">
+    <xacro:include filename="$(find zbl_arm_6a_description)/urdf/parallel_gripper.urdf.xacro" />
+    <xacro:include filename="$(find zbl_arm_6a_description)/urdf/parallel_gripper.ros2_control.xacro" />
+    <xacro:parallel_gripper prefix="arm_"
+                            use_geometry_collision="$(arg use_geometry_collision)" />
+    <joint name="gripper_connector"
+           type="fixed">
+      <parent link="arm_link6" />
+      <child link="arm_gripper_base_link" />
+      <origin xyz="0 0 0"
+              rpy="0 0 0" />
+    </joint>
+    <xacro:parallel_gripper_ros2_control name="arm_gripper"
+                                         prefix="arm_"
+                                         can_interface="$(arg can_interface)"
+                                         use_ipc="1"
+                                         mock_robot="$(arg mock_robot)" />
+  </xacro:if>
+  <xacro:if value="${gripper_type_prop == 'g'}">
+    <xacro:include filename="$(find zbl_arm_6a_description)/urdf/zbl_g1_gripper_dvt1.urdf.xacro" />
+    <xacro:include filename="$(find zbl_arm_6a_description)/urdf/zbl_g_gripper.ros2_control.xacro" />
+    <xacro:zbl_g1_gripper prefix="arm_"
+                            use_geometry_collision="$(arg use_geometry_collision)" />
+    <joint name="gripper_connector"
+           type="fixed">
+      <parent link="arm_link6" />
+      <child link="arm_gripper_base_link" />
+      <origin xyz="0 0 0"
+              rpy="0 0 0" />
+    </joint>
+    <xacro:zbl_g_gripper_ros2_control name="arm_gripper"
+                                        prefix="arm_"
+                                        can_interface="$(arg can_interface)"
+                                        use_ipc="1"
+                                        mock_robot="$(arg mock_robot)" />
+  </xacro:if>
 </robot>
